Commit message: Update Origin position
Updated the origin position, so that it maches with reality. Will be changed later, because of a new holder, which makes the use of the offset redundant

File: rtb-data/rtbdata/xacro/tm5_description/urdf/tm5_700.urdf.xacro (robot description, xacro)
@@ -338,5 +338,5 @@
       <parent link="${prefix}flange_link" />
       <child link="${prefix}tool0" />
-      <origin xyz="0 0.03 0.151" rpy="0 0 0" />
+      <origin xyz="0 0.0425 0.151" rpy="0 0 0" />
     </joint>
   </xacro:macro>

Commit message: Update of the coil holder
Updated the coil holder to match the soon to be printed holder. Also updated the urdf file of the robot

File: rtb-data/rtbdata/xacro/tm5_description/urdf/tm5_700.urdf.xacro (robot description, xacro)
@@ -338,5 +338,5 @@
       <parent link="${prefix}flange_link" />
       <child link="${prefix}tool0" />
-      <origin xyz="0 0.0425 0.151" rpy="0 0 0" />
+      <origin xyz="0 0 0.151" rpy="0 0 0" />
     </joint>
   </xacro:macro>
